File: fan_control.kicad_pcb (KiCad board)
At the start: 2 copper layers, 50 x 68.6 mm, 45 parts, among them M1 0VAC, M1 Fan, M2 +15VAC, M4 SI_B, M5 SI_B, M6 SI_E, Q10 BC557, Q11 BC557, Q12 BC557, Q13 BC557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

Commit message: progress on schematics
Parts:
- removed M1: 0VAC, Connector_PinHeader_2.54mm:PinHeader_1x02_P2.54mm_Vertical
- removed M1: Fan, Connector_PinHeader_2.54mm:PinHeader_1x02_P2.54mm_Vertical
- removed M2: +15VAC, Connector_PinHeader_2.54mm:PinHeader_1x02_P2.54mm_Vertical
- removed M4, M5: SI_B, Connector_PinHeader_2.54mm:PinHeader_1x02_P2.54mm_Vertical
- removed M6: SI_E, Connector_PinHeader_2.54mm:PinHeader_1x02_P2.54mm_Vertical
- removed Q2: IRFZ34N, Package_TO_SOT_THT:TO-220-3_Vertical
- removed R4: 50k, Resistor_THT:R_Axial_DIN0207_L6.3mm_D2.5mm_P2.54mm_Vertical
- added D4: 1N4007, Diode_THT:D_DO-41_SOD81_P2.54mm_Vertical_AnodeUp, F.Cu at (59.6, 86.4)
- added J1: Conn_01x02_Male, Connector_PinHeader_2.54mm:PinHeader_1x02_P2.54mm_Vertical, F.Cu at (74.8, 86.4)
- added J2: Conn_01x02_Male, Connector_PinHeader_2.54mm:PinHeader_1x02_P2.54mm_Vertical, F.Cu at (72.3, 55.9)
- added J3: Conn_01x02_Male, Connector_PinHeader_2.54mm:PinHeader_1x02_P2.54mm_Vertical, F.Cu at (69.7, 66.1)
- added J4: Conn_01x02_Male, Connector_PinHeader_2.54mm:PinHeader_1x02_P2.54mm_Vertical, F.Cu at (46.9, 38.1)
- added J5: Conn_01x02_Male, Connector_PinHeader_2.54mm:PinHeader_1x02_P2.54mm_Vertical, F.Cu at (52.0, 55.9)
- added J6: Conn_01x02_Male, Connector_PinHeader_2.54mm:PinHeader_1x02_P2.54mm_Vertical, F.Cu at (57.0, 88.9)
- added J7: Conn_01x02_Male, Connector_PinHeader_2.54mm:PinHeader_1x02_P2.54mm_Vertical, F.Cu at (87.5, 48.3)
- added J8: Conn_01x02_Male, Connector_PinHeader_2.54mm:PinHeader_1x02_P2.54mm_Vertical, F.Cu at (46.9, 91.5)
Connections:
- net /0VAC renamed 0VAC
- net SI_E renamed E
- net SI_F+ renamed F+
- D7 pad 2: /+15VAC -> +15VAC
- R12 pad 1: SI_C -> C
- R24 pad 1: SI_B -> B
Routing:
- net Net-(M1-Pad2): track 35.6 -> 0.00 mm
- net F+: track 43.2 -> 15.2 mm
- net +15V: track 147.3 -> 124.5 mm
- net 0: track 172.7 -> 165.1 mm
- net +15VAC: track 0.00 -> 7.62 mm
- net SI_B: track 5.08 -> 0.00 mm
- net B: track 0.00 -> 5.08 mm
- net SI_C: track 5.08 -> 0.00 mm
- net C: track 0.00 -> 5.08 mm
- net /+15VAC: track 4.34 -> 0.00 mm
